File: pcb/m68k.sch (KiCad schematic (older format))
At the start: 120 parts, among them J1 USB_B_Micro, J2 Mini-DIN-6, J4 DB15_Male_HighDensity, J5 FTSH-105-01-L-DV-K, J6 FTSH-105-01-L-DV-K, J7 FTSH-105-01-L-DV-K, J8 Micro_SD_Card, U1 93LC56, U10 25LCxxx, U11 TXB0108DQSR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

Commit message: Battle Bus
Connections:
- net ADDR_OE: now also U13.34 (IOL_25B); no longer U13.144 (IOT_222)
- net BERRn: now also U13.110 (IOT_168); no longer U13.24 (IOL_17B)
- net a1: now also U13.29 (IOL_23B); no longer U13.134 (IOT_212)
- net a10: now also U13.10 (IOL_5B); no longer U13.119 (IOT_178)
- net a11: now also U13.9 (IOL_5A); no longer U13.118 (IOT_177)
- net a12: now also U13.8 (IOL_4B); no longer U13.117 (IOT_174)
- net a13: now also U13.7 (IOL_4A); no longer U13.116 (IOT_173)
- net a14: now also U13.4 (IOL_3B); no longer U13.115 (IOT_172)
- net a15: now also U13.3 (IOL_3A); no longer U13.114 (IOT_171)
- net a16: now also U13.2 (IOL_2B); no longer U13.113 (IOT_170)
- net a17: now also U13.1 (IOL_2A); no longer U13.112 (IOT_169)
- net a18: now also U13.19 (IOL_13A); no longer U13.110 (IOT_168)
- net a19: now also U13.18 (IOL_12B); no longer U13.34 (IOL_25B)
- net a2: now also U13.28 (IOL_23A); no longer U13.130 (IOT_206)
- net a20: now also U13.12 (IOL_8B); no longer U13.33 (IOL_25A)
- net a21: now also U13.33 (IOL_25A); no longer U13.32 (IOL_24B)
- net a22: now also U13.32 (IOL_24B); no longer U13.31 (IOL_24A)
- net a23: now also U13.31 (IOL_24A); no longer U13.29 (IOL_23B)
- net a3: now also U13.26 (IOL_18B); no longer U13.129 (IOT_198_GBIN0)
- net a4: now also U13.25 (IOL_18A); no longer U13.128 (IOT_197_GBIN1)
- net a5: now also U13.24 (IOL_17B); no longer U13.125 (IOT_192)
- net a6: now also U13.23 (IOL_17A); no longer U13.124 (IOT_191)
- net a7: now also U13.22 (IOL_14B); no longer U13.122 (IOT_190)
- net a8: now also U13.20 (IOL_13B_GBIN7); no longer U13.121 (IOT_181)
- net a9: now also U13.11 (IOL_8A); no longer U13.120 (IOT_179)
- net d0: now also U13.130 (IOT_206); no longer U13.20 (IOL_13B_GBIN7)
- net d1: now also U13.129 (IOT_198_GBIN0); no longer U13.19 (IOL_13A)
- net d10: now also U13.117 (IOT_174); no longer U13.8 (IOL_4B)
- net d11: now also U13.116 (IOT_173); no longer U13.7 (IOL_4A)
- net d12: now also U13.115 (IOT_172); no longer U13.4 (IOL_3B)
- net d13: now also U13.114 (IOT_171); no longer U13.3 (IOL_3A)
- net d14: now also U13.113 (IOT_170); no longer U13.2 (IOL_2B)
- net d15: now also U13.112 (IOT_169); no longer U13.1 (IOL_2A)
- net d2: now also U13.128 (IOT_197_GBIN1); no longer U13.18 (IOL_12B)
- net d3: now also U13.125 (IOT_192); no longer U13.17 (IOL_12A)
- net d4: now also U13.124 (IOT_191); no longer U13.16 (IOL_10B)
- net d5: now also U13.122 (IOT_190); no longer U13.15 (IOL_10A)
- net d6: now also U13.121 (IOT_181); no longer U13.12 (IOL_8B)
- net d7: now also U13.120 (IOT_179); no longer U13.11 (IOL_8A)
- net d8: now also U13.119 (IOT_178); no longer U13.10 (IOL_5B)
- net d9: now also U13.118 (IOT_177); no longer U13.9 (IOL_5A)
- net at U9.28 (OE#): now also U13.134 (IOT_212); no longer U13.22 (IOL_14B)
- net at U11.1 (A1), U9.11 (WE#): now also U13.15 (IOL_10A); no longer U13.23 (IOL_17A)
- net at U11.2 (A2), U9.14 (UB#): now also U13.16 (IOL_10B); no longer U13.26 (IOL_18B)
- net at U11.3 (A3), U9.15 (LB#): now also U13.17 (IOL_12A); no longer U13.28 (IOL_23A)

Commit message: PINS
Connections:
- net d1: now also U13.128 (IOT_197_GBIN1); no longer U13.129 (IOT_198_GBIN0)
- net d10: now also U13.122 (IOT_190); no longer U13.117 (IOT_174)
- net d11: now also U13.120 (IOT_179); no longer U13.116 (IOT_173)
- net d12: now also U13.118 (IOT_177); no longer U13.115 (IOT_172)
- net d13: now also U13.116 (IOT_173); no longer U13.114 (IOT_171)
- net d14: now also U13.114 (IOT_171); no longer U13.113 (IOT_170)
- net d2: now also U13.124 (IOT_191); no longer U13.128 (IOT_197_GBIN1)
- net d3: now also U13.121 (IOT_181); no longer U13.125 (IOT_192)
- net d4: now also U13.119 (IOT_178); no longer U13.124 (IOT_191)
- net d5: now also U13.117 (IOT_174); no longer U13.122 (IOT_190)
- net d6: now also U13.115 (IOT_172); no longer U13.121 (IOT_181)
- net d7: now also U13.113 (IOT_170); no longer U13.120 (IOT_179)
- net d8: now also U13.129 (IOT_198_GBIN0); no longer U13.119 (IOT_178)
- net d9: now also U13.125 (IOT_192); no longer U13.118 (IOT_177)
Changed lines of the file:
@@
 	8550 6200 8450 6200
+Wire Wire Line
+	8450 6000 8550 6000
+Wire Wire Line
+	8550 5800 8450 5800
+Wire Wire Line
+	8450 5600 8550 5600
+Wire Wire Line
+	8550 5400 8450 5400
+Wire Wire Line
+	8450 5200 8550 5200
+Wire Wire Line
+	8550 5000 8450 5000
+Wire Wire Line
+	8450 4800 8550 4800
 Wire Wire Line
 	8450 6100 8550 6100
 Wire Wire Line
-	8550 6000 8450 6000
-Wire Wire Line
-	8450 5900 8550 5900
-Wire Wire Line
-	8550 5800 8450 5800
+	8550 5900 8450 5900
 Wire Wire Line
 	8450 5700 8550 5700
 Wire Wire Line
-	8550 5600 8450 5600
+	8550 5500 8450 5500
 Wire Wire Line
-	8450 5500 8550 5500
-Wire Wire Line
-	8450 5400 8550 5400
-Wire Wire Line
-	8550 5300 8450 5300
-Wire Wire Line
-	8450 5200 8550 5200
+	8450 5300 8550 5300
 Wire Wire Line
 	8550 5100 8450 5100
 Wire Wire Line
-	8450 5000 8550 5000
-Wire Wire Line
-	8550 4900 8450 4900
-Wire Wire Line
-	8450 4800 8550 4800
+	8450 4900 8550 4900
 Wire Wire Line
 	8550 4700 8450 4700
 Text Label 8450 4700 0    50   ~ 0
 d15
+Text Label 8450 4900 0    50   ~ 0
+d14
+Text Label 8450 5100 0    50   ~ 0
+d13
+Text Label 8450 5300 0    50   ~ 0
+d12
+Text Label 8450 5500 0    50   ~ 0
+d11
+Text Label 8450 5700 0    50   ~ 0
+d10
+Text Label 8450 5900 0    50   ~ 0
+d9
+Text Label 8450 6100 0    50   ~ 0
+d8
 Text Label 8450 4800 0    50   ~ 0
-d14
-Text Label 8450 4900 0    50   ~ 0
-d13
+d7
 Text Label 8450 5000 0    50   ~ 0
-d12
-Text Label 8450 5100 0    50   ~ 0
-d11
+d6
 Text Label 8450 5200 0    50   ~ 0
-d10
-Text Label 8450 5300 0    50   ~ 0
-d9
+d5
 Text Label 8450 5400 0    50   ~ 0
-d8
-Text Label 8450 5500 0    50   ~ 0
-d7
+d4
 Text Label 8450 5600 0    50   ~ 0
-d6
-Text Label 8450 5700 0    50   ~ 0
-d5
+d3
 Text Label 8450 5800 0    50   ~ 0
-d4
-Text Label 8450 5900 0    50   ~ 0
-d3
+d2
 Text Label 8450 6000 0    50   ~ 0
-d2
-Text Label 8450 6100 0    50   ~ 0
 d1
 Text Label 8450 6200 0    50   ~ 0
@@
 	8450 6200 8350 6300
 Entry Wire Line
+	8450 6000 8350 6100
+Entry Wire Line
+	8450 5800 8350 5900
+Entry Wire Line
+	8450 5600 8350 5700
+Entry Wire Line
+	8450 5400 8350 5500
+Entry Wire Line
+	8450 5200 8350 5300
+Entry Wire Line
+	8450 5000 8350 5100
+Entry Wire Line
+	8450 4800 8350 4900
+Entry Wire Line
 	8450 6100 8350 6200
-Entry Wire Line
-	8450 6000 8350 6100
 Entry Wire Line
 	8450 5900 8350 6000
 Entry Wire Line
-	8450 5800 8350 5900
-Entry Wire Line
 	8450 5700 8350 5800
-Entry Wire Line
-	8450 5600 8350 5700
 Entry Wire Line
 	8450 5500 8350 5600
 Entry Wire Line
-	8450 5400 8350 5500
-Entry Wire Line
 	8450 5300 8350 5400
-Entry Wire Line
-	8450 5200 8350 5300
 Entry Wire Line
 	8450 5100 8350 5200
 Entry Wire Line
-	8450 5000 8350 5100
+	8450 4700 8350 4800
 Entry Wire Line
 	8450 4900 8350 5000
-Entry Wire Line
-	8450 4700 8350 4800
-Entry Wire Line
-	8450 4800 8350 4900
 Wire Bus Line
 	7400 4800 8350 4800

Commit message: WHERE'S ROUTING?
Connections:
- net CDONE: now also U3.24 (ADBUS7); no longer U3.23 (ADBUS6)
- net CRESET_Bn: now also U3.23 (ADBUS6); no longer U3.24 (ADBUS7)
- net nHOLD: now also U13.70 (IOB_107_SCK); no longer U13.64 (IOB_104_CBSEL1)
- net at U10.5 (MOSI), U3.17 (ADBUS1): now also U13.68 (IOB_106_SDI); no longer U13.67 (IOB_105_SDO)
- net ADBUS: now reaches U10.2 (MISO), U3.18 (ADBUS2)
- net ADBUS: now also U13.64 (IOB_104_CBSEL1); no longer U13.68 (IOB_106_SDI)
- net at R8.1, U10.6 (SCK), U3.16 (ADBUS0): now also U13.71 (IOB_108_SS); no longer U13.70 (IOB_107_SCK)
- net at R10.1, U10.1 (~CS), U3.21 (ADBUS4): now also U13.67 (IOB_105_SDO); no longer U13.71 (IOB_108_SS)
Other:
- moved on the sheet: U13F
Changed lines of the file:
@@
 	8100 6200 8100 3400
 Wire Wire Line
-	5350 11800 6150 11800
+	5350 11800 6300 11800
 Wire Wire Line
 	5350 12200 5450 12200
@@
 	5350 11900 5650 11900
 Connection ~ 7050 11700
-Connection ~ 6150 11800
-Connection ~ 6050 12000
+Connection ~ 6300 11800
 Connection ~ 5950 11900
 Wire Wire Line
@@
 	7050 11650 7050 11700
 Wire Wire Line
-	6150 11650 6150 11800
+	6150 11650 6300 11800
 Wire Wire Line
 	7050 11250 7050 11300
@@
 Wire Wire Line
 	6600 11300 7050 11300
-Text GLabel 5450 12400 2    50   Input ~ 0
+Text GLabel 5450 12500 2    50   Input ~ 0
 CDONE
 Wire Wire Line
@@
 	13000 7750 13000 7800
 Wire Wire Line
-	7550 11600 7650 11600
-Wire Wire Line
-	7050 11700 7650 11700
-Wire Wire Line
-	6150 11800 7650 11800
-Wire Wire Line
-	7650 11900 5950 11900
-Wire Wire Line
-	6050 12000 7650 12000
+	7800 11900 5950 11900
 $Comp
 L m68k-rescue:iCE40-HX4K-TQ144-Lattice_iCE_FPGA U13
 U 6 1 5CE24752
-P 7650 12000
-F 0 "U13" H 8581 11853 60  0000 L CNN
-F 1 "iCE40-HX4K-TQ144" H 8581 11747 60  0000 L CNN
-F 2 "Package_QFP:TQFP-144_20x20mm_P0.5mm" H 7650 12000 50  0001 C CNN
-F 3 "" H 7650 12000 50  0001 C CNN
-	6    7650 12000
+P 8700 12000
+F 0 "U13" H 9631 11853 60  0000 L CNN
+F 1 "iCE40-HX4K-TQ144" H 9631 11747 60  0000 L CNN
+F 2 "Package_QFP:TQFP-144_20x20mm_P0.5mm" H 8700 12000 50  0001 C CNN
+F 3 "" H 8700 12000 50  0001 C CNN
+	6    8700 12000
 	1    0    0    1
 $EndComp
@@
 Text GLabel 13000 10050 0    50   BiDi ~ 0
 nWP
-Text GLabel 13000 10150 0    50   BiDi ~ 0
+Text GLabel 8700 11800 0    50   BiDi ~ 0
 nHOLD
 $Comp
@@
 Text GLabel 7600 12300 2    50   BiDi ~ 0
 nWP
-Text GLabel 5450 12500 2    50   Output ~ 0
+Text GLabel 5450 12400 2    50   Output ~ 0
 CRESET_Bn
 $Comp
@@
 	6200 12400 6050 12400
 Wire Wire Line
-	6150 12300 6150 11800
+	6150 12300 6300 11800
 Wire Wire Line
 	6200 12300 6150 12300
@@
 Wire Wire Line
 	8300 6300 8250 6300
+Wire Wire Line
+	7900 11800 7900 11700
+Wire Wire Line
+	6300 11800 7900 11800
+Wire Wire Line
+	7550 11600 8700 11600
+Wire Wire Line
+	7900 11700 8700 11700
+Text GLabel 8500 12200 2    50   Input ~ 0
+ADBUS
+Text GLabel 13000 10150 0    50   Input ~ 0
+ADBUS
+Wire Wire Line
+	7050 11700 7850 11700
+Wire Wire Line
+	7800 11900 7800 12200
+Wire Wire Line
+	7800 12200 8500 12200
+Wire Wire Line
+	7850 11700 7850 12000
+Wire Wire Line
+	7850 12000 8700 12000
+Wire Wire Line
+	6050 12000 7600 12000
+Wire Wire Line
+	7600 12000 7600 12100
+Wire Wire Line
+	7600 12100 8150 12100
+Wire Wire Line
+	8150 12100 8150 11900
+Wire Wire Line
+	8150 11900 8700 11900
+Connection ~ 6050 12000
 Wire Bus Line
 	18600 2100 18600 2800

Commit message: pcb stuff
Connections:
- net at U13.47 (IOB_79): now also J8.7 (DAT0); no longer J8.2 (DAT3/CD)
- net at U13.48 (IOB_80): now also J8.5 (CLK); no longer J8.3 (CMD)
- net at U13.49 (IOB_81_GBIN5): now also J8.3 (CMD); no longer J8.5 (CLK)
- net at U13.52 (IOB_82_GBIN4): now also J8.2 (DAT3/CD); no longer J8.7 (DAT0)
Changed lines of the file:
@@
 NoConn ~ 11300 9750
 NoConn ~ 11300 9050
-Wire Wire Line
-	11300 9650 11700 9650
 $Comp
 L power:+5V #PWR0147
@@
 	-1   0    0    -1
 $EndComp
-Wire Wire Line
-	11300 9150 13100 9150
-Wire Wire Line
-	11300 9250 13100 9250
-Wire Wire Line
-	11600 9350 13100 9350
-Wire Wire Line
-	11700 9450 13100 9450
 $Comp
 L Device:R R22
@@
 Wire Wire Line
 	11600 9450 11600 9350
-Wire Wire Line
-	11700 9650 11700 9450
 Text Label 18700 1900 0    50   ~ 0
 b0
@@
 	8150 11900 8700 11900
 Connection ~ 6050 12000
+Wire Wire Line
+	11300 9150 11850 9150
+Wire Wire Line
+	11850 9150 11850 9450
+Wire Wire Line
+	11850 9450 13100 9450
+Wire Wire Line
+	11300 9650 12050 9650
+Wire Wire Line
+	12050 9650 12050 9150
+Wire Wire Line
+	12050 9150 13100 9150
+Wire Wire Line
+	11600 9350 12150 9350
+Wire Wire Line
+	12150 9350 12150 9250
+Wire Wire Line
+	12150 9250 13100 9250
+Wire Wire Line
+	11300 9250 11950 9250
+Wire Wire Line
+	11950 9250 11950 9400
+Wire Wire Line
+	11950 9400 12250 9400
+Wire Wire Line
+	12250 9400 12250 9350
+Wire Wire Line
+	12250 9350 13100 9350
 Wire Bus Line
 	18600 2100 18600 2800

Commit message: Repin
Connections:
- net BERRn: now also U13.107 (IOR_167); no longer U13.110 (IOT_168)
- net DIR: now also U13.110 (IOT_168); no longer U13.107 (IOR_167)
Changed lines of the file:
@@
 Text GLabel 5900 6650 2    50   Input ~ 0
 DIR
-Text GLabel 18700 4000 0    50   Output ~ 0
+Text GLabel 7950 4600 0    50   Output ~ 0
 DIR
 Wire Wire Line
@@
 Wire Wire Line
 	1050 4200 1150 4200
-Text GLabel 7950 4600 0    50   Output ~ 0
+Text GLabel 18700 4000 0    50   Output ~ 0
 BERRn
 $Comp

Commit message: SRAM!!!!
Connections:
- net DATA_OEn: now also U13.135 (IOT_213); no longer U13.60 (IOB_95)
- net GND: no longer U9.26 (CE#)
- net at U11.4 (A4): now also U13.136 (IOT_214); no longer U13.135 (IOT_213)
- net at U11.7 (A5): now also U13.137 (IOT_215); no longer U13.136 (IOT_214)
- net at U11.8 (A6): now also U13.138 (IOT_216); no longer U13.137 (IOT_215)
- net at U12.1 (A1): now also U13.139 (IOT_217); no longer U13.138 (IOT_216)
- net at U12.2 (A2): now also U13.141 (IOT_219); no longer U13.139 (IOT_217)
- net at U12.3 (A3): now also U13.142 (IOT_220); no longer U13.141 (IOT_219)
- net at U12.4 (A4): now also U13.143 (IOT_221); no longer U13.142 (IOT_220)
- net at U12.7 (A5): now also U13.60 (IOB_95); no longer U13.143 (IOT_221)
- net CE#: now reaches U13.144 (IOT_222)
- net CE#: now also U9.26 (CE#)
Other:
- moved on the sheet: J2, R13, R14, U11, U12

Commit message: clean up pins
Other:
- moved on the sheet: C10, C9, R1, R10, R11, R12, R8, R9, U10, U13A, U13F, U18

Commit message: SAVE
Connections:
- net ASn: now also U11.13 (B7); no longer U12.16 (B4)
- net BGn: now also U11.16 (B4); no longer U12.20 (B1)
- net CDONE: now also U12.2 (A2); no longer U12.8 (A6)
- net E: now also U11.14 (B6); no longer U12.17 (B3)
- net FC0: now also U11.20 (B1); no longer U11.16 (B4)
- net FC1: now also U11.18 (B2); no longer U11.15 (B5)
- net FC2: now also U11.17 (B3); no longer U11.14 (B6)
- net HALTn: now also U12.20 (B1); no longer U12.15 (B5)
- net LDSn: now also U12.13 (B7); no longer U11.17 (B3)
- net PS2_CLK: now also U12.4 (A4); no longer U12.10 (A8)
- net PS2_DATA: now also U12.3 (A3); no longer U12.9 (A7)
- net RESETn: now also U12.18 (B2); no longer U12.14 (B6)
- net R_Wn: now also U12.15 (B5); no longer U11.20 (B1)
- net UDSn: now also U12.14 (B6); no longer U11.18 (B2)
- net VMAn: now also U11.15 (B5); no longer U12.18 (B2)
- net at U13.136 (IOT_214): now also U11.1 (A1); no longer U11.4 (A4)
- net at U13.137 (IOT_215): now also U11.2 (A2); no longer U11.7 (A5)
- net at U13.138 (IOT_216): now also U11.3 (A3); no longer U11.8 (A6)
- net at U13.139 (IOT_217): now also U11.4 (A4); no longer U12.1 (A1)
- net at U13.141 (IOT_219): now also U11.7 (A5); no longer U12.2 (A2)
- net at U13.142 (IOT_220): now also U11.8 (A6); no longer U12.3 (A3)
- net at U13.143 (IOT_221): now also U11.9 (A7); no longer U12.4 (A4)
- net at U13.60 (IOB_95): now also U12.1 (A1); no longer U12.7 (A5)
- net at U13.15 (IOL_10A), U9.11 (WE#): now also U12.7 (A5); no longer U11.1 (A1)
- net at U13.16 (IOL_10B), U9.14 (UB#): now also U12.8 (A6); no longer U11.2 (A2)
- net at U13.17 (IOL_12A), U9.15 (LB#): now also U12.9 (A7); no longer U11.3 (A3)
- net at J2.1, R14.2: now also U12.17 (B3); no longer U12.13 (B7)
- net at J2.5, R13.2: now also U12.16 (B4); no longer U12.12 (B8)
Other:
- moved on the sheet: J2, R13, R14, U11
